Commit message: fix(g1_description): adjust Gazebo plugin z_offset to -0.82 for correct ground alignment

File: src/g1_description/urdf/g1_29dof.urdf (robot description, URDF)
Before this commit: robot g1_29dof, 40 links, 39 joints
Links:
- added link base_footprint
- added link base_link_nav
Joints:
- added joint base_footprint_to_base_link_nav: type fixed, parent base_footprint, child base_link_nav, origin xyz=0 0 0 rpy=0 0 0
- added joint base_footprint_to_pelvis: type fixed, parent base_footprint, child pelvis, origin xyz=0 0 0.92 rpy=0 0 0
